File: kicad/keychain.kicad_sch (KiCad schematic)
At the start: 53 parts, among them J1 OLED 1.5in SSD1327, J2 LiPo 3.7V, J3 USB-C, SW1 USER1, SW2 USER2, SW3 PWR, SW4 BOOT, SW5 RST, U1 ESP32-C6-MINI-1, U2 MCP73831, U3 AP2112K-3.3, U4 TLV61046A, U5 74AHCT1G125, U6 ESDA6V1-5SC6

Commit message: Schematic: ESP32-C6 + 2.36in e-Paper(G) FPC + SK6812 x4 + LiPo
Replace OLED design with e-paper badge: FH12-26S FPC connector with
discrete boost drive (NMOS/inductor/diodes/caps), SK6812s on switched
VBAT, minimal USB-C (5.1k CC only), MCP73831, AP2112K, power switch,
BOOT + USER buttons. Single A3 sheet, net labels and power symbols
with short stubs, ERC-clean.

Generated with [Devin](https://devin.ai)

Co-Authored-By: Devin <158243242+devin-ai-integration[bot]@users.noreply.github.com>
Parts:
- removed D1: SMAJ5.0A, Diode_SMD:D_SMA, symbol Diode:SMAJ5.0A
- removed F1: 0.5A, Resistor_SMD:R_1206_3216Metric, symbol Device:Polyfuse
- removed J1: OLED 1.5in SSD1327, Connector_PinHeader_2.54mm:PinHeader_1x07_P2.54mm_Vertical, symbol Connector_Generic:Conn_01x07
- removed J3: USB-C, Connector_USB:USB_C_Receptacle_HRO_TYPE-C-31-M-12, symbol Connector:USB_C_Receptacle_USB2.0_16P
- removed LED1: RED, LED_SMD:LED_0603_1608Metric, symbol Device:LED
- removed LED2: GRN, LED_SMD:LED_0603_1608Metric, symbol Device:LED
- removed LED5, LED6: SK6812MINI, LED_SMD:LED_SK6812MINI_PLCC4_3.5x3.5mm_P1.75mm, symbol LED:SK6812MINI
- removed R10, R13, R9: 100k, Resistor_SMD:R_0603_1608Metric, symbol Device:R
- removed R11: 510k, Resistor_SMD:R_0603_1608Metric, symbol Device:R
- removed R12: 97.6k, Resistor_SMD:R_0603_1608Metric, symbol Device:R
- removed R14: 330, Resistor_SMD:R_0603_1608Metric, symbol Device:R
- removed R15: 1k, Resistor_SMD:R_0603_1608Metric, symbol Device:R
- removed SW1: USER1, Button_Switch_SMD:SW_Push_1P1T_XKB_TS-1187A, symbol Switch:SW_Push
- removed SW3: PWR, Button_Switch_SMD:SW_SPDT_Shouhan_MSK12C02, symbol Switch:SW_SPDT
- removed SW4: BOOT, Button_Switch_SMD:SW_Push_1P1T_XKB_TS-1187A, symbol Switch:SW_Push
- removed SW5: RST, Button_Switch_SMD:SW_Push_1P1T_XKB_TS-1187A, symbol Switch:SW_Push
- removed U4: TLV61046A, Package_TO_SOT_SMD:SOT-23-6, symbol Regulator_Switching:TLV61046ADB
- removed U5: 74AHCT1G125, Package_TO_SOT_SMD:SOT-23-5, symbol 74xGxx:74AHCT1G125
- removed U6: ESDA6V1-5SC6, Package_TO_SOT_SMD:SOT-23-6, symbol Power_Protection:ESDA6V1-5SC6
- added C15, C16, C17, C18: 100nF, Capacitor_SMD:C_0603_1608Metric, symbol Device:C
- added D1, D2, D3: SS34, Diode_SMD:D_SMA, symbol Device:D_Schottky
- added J1: USB-C, Connector_USB:USB_C_Receptacle_HRO_TYPE-C-31-M-12, symbol Connector:USB_C_Receptacle_USB2.0_16P
- added J3: EPD FPC, Connector_FFC-FPC:Hirose_FH12-26S-0.5SH_1x26-1MP_P0.50mm_Horizontal, symbol Connector_Generic:Conn_01x26
- added LED1, LED2: SK6812MINI, LED_SMD:LED_SK6812MINI_PLCC4_3.5x3.5mm_P1.75mm, symbol LED:SK6812MINI
- added Q1: SI1304BDL, Package_TO_SOT_SMD:SOT-23, symbol Device:Q_NMOS
- added SW1: PWR, Button_Switch_SMD:SW_SPDT_Shouhan_MSK12C02, symbol Switch:SW_SPDT
- added SW3: USER, Button_Switch_SMD:SW_Push_1P1T_XKB_TS-1187A, symbol Switch:SW_Push
- C10, C11, C12, C13, C14: value 100nF -> 1uF
- C8, C9: value 10uF -> 1uF
- J2: value LiPo 3.7V -> LiPo
- L1: value 2.2uH -> 47uH
- R3: value 22 -> 4.7k
- R4: value 22 -> 10k
- R5: value 4.7k -> 10k
- R6: value 1k -> 10k
- R7: value 10k -> 100k
- R8: value 10k -> 1
- SW2: value USER2 -> BOOT
- U1: footprint RF_Module:ESP32-C6-MINI-1 -> keychain:ESP32-C6-MINI-1
Connections:
- net CHG_LED is gone; now on net +3V3: R6.1
- net LED_D0 is gone; now on net LED_C2: LED3.3 (DIN)
- net USB_DM_CONN is gone; now on net +3V3: R4.1
- net USB_DP_CONN is gone; now on net PROG: R3.1
- net VBUS_F is gone; now on net VBUS: U2.4 (V_{DD})
- net +3V3: now also C6.1, C8.1, L1.1, R5.1, J3.10 (Pin_10), J3.12 (Pin_12), J3.13 (Pin_13); no longer C14.1, R7.1, R8.1
- net CC1: now also J1.A5 (CC1)
- net CC2: now also J1.B5 (CC2)
- net EN: now also C7.1, R4.2; no longer C6.1, R7.2
- net GND: now also R3.2, R7.2, R8.2, C15.2, C16.2, C17.2, C18.2, D2.1 (K), J1.A1 (GND), J1.A12 (GND), J1.B1 (GND), J1.B12 (GND), J1.SH (SHIELD), J3.14 (Pin_14), J3.25 (Pin_25), J3.8 (Pin_8), J3.9 (Pin_9), LED1.2 (VSS), LED2.2 (VSS), SW3.2; no longer C9.2, R5.2, R6.2
- net LED_C1: now also LED1.1 (DOUT), LED2.3 (DIN); no longer LED3.1 (DOUT), LED4.3 (DIN)
- net LED_C2: now also LED2.1 (DOUT); no longer LED4.1 (DOUT)
- net LED_C3: now also LED3.1 (DOUT), LED4.3 (DIN)
- net LED_DIN: now also U1.5 (IO2), LED1.3 (DIN)
- net PROG: no longer R5.1
- net USB_DM: now also J1.A7 (D-), J1.B7 (D-); no longer R4.2
- net USB_DP: now also J1.A6 (D+), J1.B6 (D+); no longer R3.2
- net VBUS: now also J1.A4 (VBUS), J1.A9 (VBUS), J1.B4 (VBUS), J1.B9 (VBUS)
- net EPD_CS: now reaches U1.26 (IO20)
- net EPD_CS: now also J3.4 (Pin_4)
- net EPD_DC: now reaches U1.27 (IO21)
- net EPD_DC: now also J3.3 (Pin_3)
- net EPD_RST: now reaches U1.28 (IO22)
- net EPD_RST: now also J3.2 (Pin_2)
- net EPD_BUSY: now reaches U1.29 (IO23)
- net EPD_BUSY: now also J3.1 (Pin_1)
- removed net +5V: C10.1, C11.1, C12.1, C13.1, C9.1, LED3.4 (VDD), LED4.4 (VDD)
- removed net BAT_ADC: C7.1, U1.5 (IO2)
- net BOOST_EN renamed EPD_DIN
- net EPD_DIN: now also J3.6 (Pin_6)
- net BOOST_SW renamed EPD_LX
- net EPD_LX: now also C9.1, D1.2 (A), Q1.D
- net BOOT renamed BTN_BOOT
- net BTN_BOOT: now also R5.2, SW2.1; no longer R8.2
- net CHG_STAT: no longer names the net of U2.1 (STAT)
- net CHG_STAT: no longer U1.19 (IO14)
- net LED_DAT_3V renamed EPD_SCK
- net EPD_SCK: now also J3.5 (Pin_5)
- net OLED_CS: no longer names the net of U1.10 (IO5)
- net OLED_DC: no longer names the net of U1.9 (IO4)
- net OLED_MOSI: no longer names the net of U1.16 (IO7)
- net OLED_RES: no longer names the net of U1.6 (IO3)
- net OLED_SCK: no longer names the net of U1.15 (IO6)
- net USER1 renamed BTN_USER
- net BTN_USER: now also R6.2, SW3.1
- net USER2: no longer names the net of U1.13 (IO1)
- net USER2: no longer SW2.1
- net VBAT renamed +BATT
- net +BATT: now also SW1.1 (A)
- net VBAT_SYS renamed VBAT_SW
- net VBAT_SW: now also LED3.4 (VDD), LED4.4 (VDD), C15.1, C16.1, C17.1, C18.1, LED1.4 (VDD), LED2.4 (VDD), SW1.2 (B); no longer C8.1, L1.1
- new net EPD_CP: C9.2, D2.2 (A), D3.1 (K)
- new net EPD_GDR: J3.15 (Pin_15), Q1.G, R7.1
- new net EPD_RESE: J3.16 (Pin_16), Q1.S, R8.1
- new net EPD_VCOM: C14.1, J3.21 (Pin_21)
- new net EPD_VGH: C10.1, D1.1 (K), J3.18 (Pin_18)
- new net EPD_VGL: C11.1, D3.2 (A), J3.17 (Pin_17)
- new net EPD_VSH: C12.1, J3.19 (Pin_19)
- new net EPD_VSL: C13.1, J3.20 (Pin_20)
- no-connect marks 21 -> 30
Other:
- note removed: "5V BOOST + LEVEL SHIFT"
- note removed: "ADDRESSABLE RGB LEDs (x4)"
- note removed: "KEYRING HOLE (GND pad)"
- note removed: "LiPo CHARGER MCP73831 (I=~215mA)"
- note removed: "MCU ESP32-C6-MINI-1 (BLE/WiFi6/USB)"
- note removed: "OLED 1.5in SSD1327 128x128 SPI"
- note removed: "PWR SWITCH + 3V3 LDO"
- note removed: "USB-C INPUT + PROTECTION"
- title: PCB Keychain - BLE OLED badge -> PCB Keychain - BLE e-Paper badge

Commit message: Fix e-paper section to match official Waveshare docs
The interim schematic guessed the FPC pinout and used a simplified
drive circuit. Rewired per the official 2.36in e-Paper (G) panel spec
and Waveshare reference module schematic: correct 26-pin mapping,
exact boost/charge-pump topology and values, BS0 tied high for 4-wire
SPI, AO3401+S8050 VCC power-gate network, all rail capacitors, and a
local FH34SRJ-26S-0.5SH footprint (datasheet connector) replacing the
FH12 footprint. Button pull-ups removed (ESP32 internal pull-ups).

Generated with [Devin](https://devin.ai)

Co-Authored-By: Devin <158243242+devin-ai-integration[bot]@users.noreply.github.com>
Parts:
- removed D1, D2, D3: SS34, Diode_SMD:D_SMA, symbol Device:D_Schottky
- removed Q1: SI1304BDL, Package_TO_SOT_SMD:SOT-23, symbol Device:Q_NMOS
- added C19, C20, C21, C22, C24, C25, C26: 1uF, Capacitor_SMD:C_0603_1608Metric, symbol Device:C
- added C23: 1.8uF, Capacitor_SMD:C_0603_1608Metric, symbol Device:C
- added C27: 10uF, Capacitor_SMD:C_0603_1608Metric, symbol Device:C
- added C28: 4.7uF, Capacitor_SMD:C_0603_1608Metric, symbol Device:C
- added C29: 100nF, Capacitor_SMD:C_0603_1608Metric, symbol Device:C
- added D1, D2, D3: MBR0530, Diode_SMD:D_SOD-123, symbol Diode:MBR0530
- added Q1: BSS138, Package_TO_SOT_SMD:SOT-23, symbol Transistor_FET:BSS138
- added Q2: AO3401A, Package_TO_SOT_SMD:SOT-23, symbol Transistor_FET:AO3401A
- added Q3: S8050, Package_TO_SOT_SMD:SOT-23, symbol Transistor_BJT:Q_NPN_BEC
- added R10, R13, R9: 47k, Resistor_SMD:R_0603_1608Metric, symbol Device:R
- added R11: 10k, Resistor_SMD:R_0603_1608Metric, symbol Device:R
- added R12: 1k, Resistor_SMD:R_0603_1608Metric, symbol Device:R
- C10, C11, C8, C9: value 1uF -> 100nF
- C12: value 1uF -> 4.7uF
- C15: value 100nF -> 4.7uF
- C16, C17, C18: value 100nF -> 1uF
- J3: footprint Connector_FFC-FPC:Hirose_FH12-26S-0.5SH_1x26-1MP_P0.50mm_Horizontal -> keychain:Hirose_FH34SRJ-26S-0.5SH_1x26-1MP_P0.50mm_Horizontal
- L1: value 47uH -> 10uH; footprint Inductor_SMD:L_1008_2520Metric -> Inductor_SMD:L_0805_2012Metric
- R5: value 10k -> 1M
- R6: value 10k -> 0.2
- R7: value 100k -> 5M
- R8: value 1 -> 100k
Connections:
- net EPD_RESE is gone; now on net GND: J3.16 (Pin_16), R8.1
- net +3V3: now also C4.2, C5.2, C6.2, R4.2, C29.2, Q2.2 (S), R9.2; no longer C4.1, C5.1, C6.1, C8.1, J3.10 (Pin_10), J3.12 (Pin_12), J3.13 (Pin_13), L1.1, R4.1, R5.1, R6.1
- net +BATT: now also C2.2; no longer C2.1
- net BTN_BOOT: no longer R5.2
- net BTN_USER: no longer R6.2
- net CC1: now also R1.2; no longer R1.1
- net CC2: now also R2.2; no longer R2.1
- net EN: now also C7.2, R4.1; no longer C7.1, R4.2
- net EPD_BUSY: now also J3.8 (Pin_8); no longer J3.1 (Pin_1)
- net EPD_CP: now also C12.1, D2.2 (A), D3.1 (K); no longer C9.2
- net EPD_CS: now also J3.11 (Pin_11); no longer J3.4 (Pin_4)
- net EPD_DC: now also J3.10 (Pin_10); no longer J3.3 (Pin_3)
- net EPD_DIN: now also J3.13 (Pin_13); no longer J3.6 (Pin_6)
- net EPD_GDR: now also J3.1 (Pin_1), J3.2 (Pin_2), R5.2, Q1.1 (G); no longer J3.15 (Pin_15), R7.1
- net EPD_LX: now also C12.2, L1.1, D1.2 (A), Q1.3 (D); no longer C9.1, L1.2
- net EPD_RST: now also J3.9 (Pin_9), R11.2, R12.2; no longer J3.2 (Pin_2)
- net EPD_SCK: now also J3.12 (Pin_12); no longer J3.5 (Pin_5)
- net EPD_VCOM: now also J3.26 (Pin_26), R7.2, C23.2; no longer C14.1, J3.21 (Pin_21)
- net EPD_VGH: now also C13.2, C14.2, J3.23 (Pin_23), D1.1 (K); no longer C10.1, J3.18 (Pin_18)
- net EPD_VGL: now also C15.2, C16.2, J3.25 (Pin_25), D3.2 (A); no longer C11.1, J3.17 (Pin_17)
- net EPD_VSH: now also J3.24 (Pin_24), C22.2; no longer C12.1, J3.19 (Pin_19)
- net EPD_VSL: now also J3.19 (Pin_19), C19.2; no longer C13.1, J3.20 (Pin_20)
- net GND: now also C1.1, C10.1, C11.1, C14.1, C15.1, C16.1, C17.1, C18.1, C2.1, C3.1, C4.1, C5.1, C6.1, C7.1, C8.1, C9.1, R1.1, R2.1, R3.1, R5.1, R6.1, R7.1, C19.1, C20.1, C21.1, C22.1, C23.1, C24.1, C25.1, C26.1, C27.1, C28.1, C29.1, Q3.2 (E); no longer C1.2, C10.2, C11.2, C12.2, C13.2, C14.2, C15.2, C16.2, C17.2, C18.2, C2.2, C3.2, C4.2, C5.2, C6.2, C7.2, C8.2, J3.14 (Pin_14), J3.25 (Pin_25), J3.8 (Pin_8), J3.9 (Pin_9), LED1.2 (VSS), LED2.2 (VSS), LED3.2 (VSS), LED4.2 (VSS), R1.2, R2.2, R3.2, R7.2, R8.2
- net PROG: now also R3.2; no longer R3.1
- net VBAT_SW: now also C10.2, C11.2, C3.2, C8.2, C9.2; no longer C15.1, C16.1, C17.1, C18.1, C3.1
- net VBUS: now also C1.2; no longer C1.1
- net EPD_EN: now reaches U1.15 (IO6)
- net EPD_EN: now also R8.2, R12.1, R13.1
- net EPD_VSHV: now reaches J3.22 (Pin_22)
- net EPD_VSHV: now also C21.2
- net VCC: now reaches J3.7 (Pin_7)
- net VCC: now also J3.14 (Pin_14), J3.15 (Pin_15), L1.2, C26.2, C27.2, C28.2, Q2.3 (D)
- new net EPD_1V8: C25.2, J3.4 (Pin_4)
- new net EPD_CPN: C13.1, D2.1 (K)
- new net EPD_GATE: Q2.1 (G), Q3.3 (C), R9.1
- new net EPD_GB: Q3.1 (B), R10.2, R11.1
- new net EPD_GC: R10.1, R13.2
- new net EPD_SNS: Q1.2 (S), R6.2
- new net EPD_TVCOM: C24.2, J3.3 (Pin_3)
- new net EPD_VSH2: C20.2, J3.21 (Pin_21)
- new net EPD_VSL2: C17.2, J3.17 (Pin_17)
- new net EPD_VSLV: C18.2, J3.18 (Pin_18)
Other:
- moved on the sheet: C1, C2, C3, C4, C5, C6, C7, J1, J2, R1, R2, R3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

Commit message: Fix netlist-review bugs in e-paper keychain schematic
- Connect all four SK6812MINI VSS pins to GND (were unconnected)
- J3 pin 1 is NC per panel spec; only pin 2 carries GDR
- Simplify VCC power gate: EPD_EN ->10k-> Q3 base, 47k base
  pull-down, Q3 collector -> Q2 gate, 47k gate pull-up to +3V3;
  EPD_RST now only U1.28 <-> J3.9; leftover resistors removed
- Charge pump: D2 cathode to GND per Waveshare reference;
  stray VGH-side pump cap removed
- Add 10k pull-up on IO8 strapping pin

ERC clean: 0 errors, 0 warnings.

Generated with [Devin](https://devin.ai)

Co-Authored-By: Devin <158243242+devin-ai-integration[bot]@users.noreply.github.com>
Parts:
- removed C13: 1uF, Capacitor_SMD:C_0603_1608Metric, symbol Device:C
- removed R12: 1k, Resistor_SMD:R_0603_1608Metric, symbol Device:R
- removed R13: 47k, Resistor_SMD:R_0603_1608Metric, symbol Device:R
- R8: value 100k -> 10k
Connections:
- net EPD_CPN is gone; now on net GND: D2.1 (K)
- net EPD_GC is gone; now on net GND: R10.1
- net +3V3: now also R11.2
- net EPD_GB: now also R8.1; no longer R11.1
- net EPD_GDR: no longer J3.1 (Pin_1)
- net EPD_RST: no longer R11.2
- net GND: now also LED1.2 (VSS), LED2.2 (VSS), LED3.2 (VSS), LED4.2 (VSS); no longer R8.1
- net IO8: now reaches U1.22 (IO8)
- net IO8: now also R11.1
- no-connect marks 30 -> 26

Commit message: Simplify schematic: ESP32-C3 SuperMini + e-paper + SK6812 x4 + TP4056
Generated with [Devin](https://devin.ai)

Co-Authored-By: Devin <158243242+devin-ai-integration[bot]@users.noreply.github.com>
Parts:
- removed C10, C11, C29, C7, C8, C9: 100nF, Capacitor_SMD:C_0603_1608Metric, symbol Device:C
- removed C12, C15, C28: 4.7uF, Capacitor_SMD:C_0603_1608Metric, symbol Device:C
- removed C14, C16, C17, C18, C19, C20, C21, C22, C24, C25, C26: 1uF, Capacitor_SMD:C_0603_1608Metric, symbol Device:C
- removed C23: 1.8uF, Capacitor_SMD:C_0603_1608Metric, symbol Device:C
- removed C27: 10uF, Capacitor_SMD:C_0603_1608Metric, symbol Device:C
- removed D1, D2, D3: MBR0530, Diode_SMD:D_SOD-123, symbol Diode:MBR0530
- removed H1: Keyring, MountingHole:MountingHole_3.2mm_M3_Pad, symbol Device:MountingHole_Pad
- removed J1: USB-C, Connector_USB:USB_C_Receptacle_HRO_TYPE-C-31-M-12, symbol Connector:USB_C_Receptacle_USB2.0_16P
- removed J2: LiPo, Connector_JST:JST_PH_S2B-PH-K_1x02_P2.00mm_Horizontal, symbol Connector_Generic:Conn_01x02
- removed J3: EPD FPC, keychain:Hirose_FH34SRJ-26S-0.5SH_1x26-1MP_P0.50mm_Horizontal, symbol Connector_Generic:Conn_01x26
- removed L1: 10uH, Inductor_SMD:L_0805_2012Metric, symbol Device:L
- removed LED1, LED2, LED3, LED4: SK6812MINI, LED_SMD:LED_SK6812MINI_PLCC4_3.5x3.5mm_P1.75mm, symbol LED:SK6812MINI
- removed Q1: BSS138, Package_TO_SOT_SMD:SOT-23, symbol Transistor_FET:BSS138
- removed Q2: AO3401A, Package_TO_SOT_SMD:SOT-23, symbol Transistor_FET:AO3401A
- removed Q3: S8050, Package_TO_SOT_SMD:SOT-23, symbol Transistor_BJT:Q_NPN_BEC
- removed R10, R9: 47k, Resistor_SMD:R_0603_1608Metric, symbol Device:R
- removed R11, R4, R8: 10k, Resistor_SMD:R_0603_1608Metric, symbol Device:R
- removed R2: 5.1k, Resistor_SMD:R_0603_1608Metric, symbol Device:R
- removed R3: 4.7k, Resistor_SMD:R_0603_1608Metric, symbol Device:R
- removed R5: 1M, Resistor_SMD:R_0603_1608Metric, symbol Device:R
- removed R6: 0.2, Resistor_SMD:R_0603_1608Metric, symbol Device:R
- removed R7: 5M, Resistor_SMD:R_0603_1608Metric, symbol Device:R
- removed SW2: BOOT, Button_Switch_SMD:SW_Push_1P1T_XKB_TS-1187A, symbol Switch:SW_Push
- removed SW3: USER, Button_Switch_SMD:SW_Push_1P1T_XKB_TS-1187A, symbol Switch:SW_Push
- removed U1: ESP32-C6-MINI-1, keychain:ESP32-C6-MINI-1, symbol RF_Module:ESP32-C6-MINI-1
- removed U2: MCP73831, Package_TO_SOT_SMD:SOT-23-5, symbol Battery_Management:MCP73831-2-OT
- removed U3: AP2112K-3.3, Package_TO_SOT_SMD:SOT-23-5, symbol Regulator_Linear:AP2112K-3.3
- added D1, D2, D3, D4: SK6812MINI, LED_SMD:LED_SK6812MINI_PLCC4_3.5x3.5mm_P1.75mm, symbol LED:SK6812MINI
- added D5: SS14, Diode_SMD:D_SMA, symbol Device:D_Schottky
- added J1: EPAPER, Connector_PinHeader_2.54mm:PinHeader_1x08_P2.54mm_Vertical, symbol Connector:Conn_01x08_Pin
- added J2: SuperMini-L, Connector_PinHeader_2.54mm:PinHeader_1x08_P2.54mm_Vertical, symbol Connector:Conn_01x08_Pin
- added J3: SuperMini-R, Connector_PinHeader_2.54mm:PinHeader_1x08_P2.54mm_Vertical, symbol Connector:Conn_01x08_Pin
- added J4: BATTERY, Connector_JST:JST_PH_B2B-PH-K_1x02_P2.00mm_Vertical, symbol Connector:Conn_01x02_Pin
- added U1: TP4056, Package_SO:SOIC-8-1EP_3.9x4.9mm_P1.27mm_EP2.29x3mm, symbol Battery_Management:TP4056-42-ESOP8
- C2: value 4.7uF -> 10uF
- C3: value 1uF -> 100nF
- C4, C5: value 10uF -> 100nF
- R1: value 5.1k -> 1.2k
- SW1: value PWR -> SW_SPDT; footprint Button_Switch_SMD:SW_SPDT_Shouhan_MSK12C02 -> Button_Switch_SMD:SW_SPDT_PCM12
Connections:
- net +BATT is gone; now on net +5V: C2.2, SW1.1 (A)
- net CC1 is gone; now on net +5V: R1.2
- net GND is gone; now on net +5V: C1.1, C2.1, C3.1, C4.1, C5.1, C6.1, R1.1
- net VBAT_SW is gone; now on net +5V: C3.2, SW1.2 (B)
- net VBUS is gone; now on net +5V: C1.2
- net EPD_BUSY: now also J1.8 (Pin_8), J2.5 (Pin_5)
- net EPD_CS: now also J1.5 (Pin_5), J3.3 (Pin_3)
- net EPD_DC: now also J1.6 (Pin_6), J3.1 (Pin_1)
- net EPD_RST: now also J1.7 (Pin_7), J3.6 (Pin_6)
- net +3V3 renamed +5V
- net +5V: now also D1.2 (VSS), D1.4 (VDD), D2.2 (VSS), D2.4 (VDD), D3.2 (VSS), D3.4 (VDD), D4.2 (VSS), D4.4 (VDD), D5.1 (K), D5.2 (A), J1.2 (Pin_2), J2.1 (Pin_1), J2.2 (Pin_2), J4.1 (Pin_1), J4.2 (Pin_2), U1.1 (TEMP), U1.2 (PROG), U1.3 (GND), U1.4 (V_{CC}), U1.5 (BAT), U1.8 (CE), U1.9 (EPAD)
- new net +3.3V: J1.1 (Pin_1), J2.3 (Pin_3)
- new net D1_DO: D1.1 (DOUT), D2.3 (DIN)
- new net D2_DO: D2.1 (DOUT), D3.3 (DIN)
- new net D3_DO: D3.1 (DOUT), D4.3 (DIN)
- new net D4_DO: D4.1 (DOUT)
- new net EPD_CLK: J1.4 (Pin_4), J2.4 (Pin_4)
- new net EPD_MOSI: J1.3 (Pin_3), J3.2 (Pin_2)
- new net LED_DATA: D1.3 (DIN), J2.6 (Pin_6)
- no-connect marks 26 -> 9
Other:
- title: PCB Keychain - BLE e-Paper badge -> PCB Keychain - ESP32-C3 e-Paper badge
