File: kicad/keychain.kicad_pcb (KiCad board)
At the start: 2 copper layers, 68 x 38 mm, 19 parts, among them J1 EPAPER, J2 SuperMini-L, J3 SuperMini-R, J4 BATTERY, SW1 SW_SPDT, U1 TP4056

Commit message: Fabrication files (DRC clean)
Parts:
- moved R1 6.32 mm to (23.0, 26.5)
- moved SW1 4.00 mm to (20.0, 33.5)
- moved C5 3.54 mm to (55.5, 35.5)
- moved U1 2.24 mm to (33.0, 29.5)
- moved J4 2.00 mm to (12.0, 33.0)
Routing:
- net D3_DO: track 62.3 -> 72.8 mm
- net GND: track 175.9 -> 166.4 mm, vias 18 -> 8
- net VBAT_SW: track 103.8 -> 112.9 mm, vias 4 -> 6
- net EPD_BUSY: track 18.4 -> 24.4 mm
- net VBAT: track 33.1 -> 39.0 mm, vias 2 -> 0
- net EPD_CLK: track 22.1 -> 27.4 mm, vias 1 -> 0
- net PROG: track 11.8 -> 17.0 mm
- net EPD_RST: track 38.1 -> 35.9 mm
- net EPD_DC: track 24.7 -> 22.7 mm
- net +3.3V: track 27.2 -> 28.8 mm, vias 1 -> 0
- net EPD_MOSI: track 34.8 -> 33.2 mm
- net D2_DO: track 10.3 -> 11.8 mm
- net D1_DO: track 86.8 -> 85.4 mm
- net EPD_CS: track 32.4 -> 31.7 mm
- net +5V: track 55.1 -> 54.5 mm, vias 4 -> 3
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